Commit message: comentario

File: src/mastering_ros_robot_description_pkg-master/urdf/ejerci5_1.urdf (robot description, URDF)
Before this commit: robot pan_tilt, 3 links, 2 joints
Links:
- added link tilt_link12, mass 1; collision cylinder length=0.4 radius=0.08; visual cylinder length=0.6 radius=0.04
Joints:
- added joint tilt_joint12: type revolute, parent tilt_link, child tilt_link12, origin xyz=0 0 0.2, axis 0 1 0, limit lower=-4.64 upper=-1.5 effort=300 velocity=0.1
- joint pan_joint: axis 0 0 1 -> 0 1 0
